Commit message: Added Moveit config files, new alias to run 'labrob_launch' & 'labrob_rviz' and changed URDF files

File: labrob/labrob_desc/urdf/rascl.urdf (robot description, URDF)
Before this commit: robot pacr, 9 links, 8 joints
Joints:
- joint shoulder_joint: limit lower=-1.570796327 upper=1.570796327 effort=100 velocity=100 -> lower=-1.5708 upper=1.5708 effort=100 velocity=100; origin xyz=0 0 0.057441 rpy=0 0 0 -> xyz=0 0 0.05744 rpy=0 0 0

File: labrob/labrob_desc/urdf/rascl2.urdf (robot description, URDF)
Before this commit: robot pacr, 9 links, 8 joints
Links:
- link base_link: geometry collision mesh filename=package://labrob_desc/meshes/base_link.stl; visual mesh filename=package://labrob_desc/meshes/base_link.dae
- link left_jaw: geometry collision mesh filename=package://labrob_desc/meshes/Hand.stl scale=1 1 1; visual mesh filename=package://labrob_desc/meshes/Hand.stl scale=1 1 1
- link lower_arm: geometry collision mesh filename=package://labrob_desc/meshes/lowerarm.stl; visual mesh filename=package://labrob_desc/meshes/lowerarm.dae
- link pinion_gear: geometry collision mesh filename=package://labrob_desc/meshes/Spur_gear__18_teeth_.stl scale=1 1 1; visual mesh filename=package://labrob_desc/meshes/Spur_gear__18_teeth_.stl scale=1 1 1
- link right_jaw: geometry collision mesh filename=package://labrob_desc/meshes/Hand.stl scale=1 1 1; visual mesh filename=package://labrob_desc/meshes/Hand.stl scale=1 1 1
- link shoulder: geometry collision mesh filename=package://labrob_desc/meshes/shoulder.dae; visual mesh filename=package://labrob_desc/meshes/shoulder.dae
- link upper_arm: geometry collision mesh filename=package://labrob_desc/meshes/upperarm.stl; visual mesh filename=package://labrob_desc/meshes/upperarm.dae
Joints:
- joint shoulder_joint: limit lower=-1.570796327 upper=1.570796327 effort=100 velocity=100 -> lower=-1.5708 upper=1.5708 effort=100 velocity=100; origin xyz=0 0 0.057441 rpy=0 0 0 -> xyz=0 0 0.05744 rpy=0 0 0

File: labrob/labrob_moveit_config/config/rascl/rascl.urdf (robot description, URDF)
Before this commit: robot pacr, 9 links, 8 joints
Links:
- link base_link: geometry collision mesh filename=package://labrob_desc/meshes/base_link.stl; visual mesh filename=package://labrob_desc/meshes/base_link.dae
- link left_jaw: geometry collision mesh filename=package://labrob_desc/meshes/Hand.stl scale=1 1 1; visual mesh filename=package://labrob_desc/meshes/Hand.stl scale=1 1 1
- link lower_arm: geometry collision mesh filename=package://labrob_desc/meshes/lowerarm.stl; visual mesh filename=package://labrob_desc/meshes/lowerarm.dae
- link pinion_gear: geometry collision mesh filename=package://labrob_desc/meshes/Spur_gear__18_teeth_.stl scale=1 1 1; visual mesh filename=package://labrob_desc/meshes/Spur_gear__18_teeth_.stl scale=1 1 1
- link right_jaw: geometry collision mesh filename=package://labrob_desc/meshes/Hand.stl scale=1 1 1; visual mesh filename=package://labrob_desc/meshes/Hand.stl scale=1 1 1
- link shoulder: geometry collision mesh filename=package://labrob_desc/meshes/shoulder.dae; visual mesh filename=package://labrob_desc/meshes/shoulder.dae
- link upper_arm: geometry collision mesh filename=package://labrob_desc/meshes/upperarm.stl; visual mesh filename=package://labrob_desc/meshes/upperarm.dae
Joints:
- joint shoulder_joint: limit lower=-1.570796327 upper=1.570796327 effort=100 velocity=100 -> lower=-1.5708 upper=1.5708 effort=100 velocity=100; origin xyz=0 0 0.057441 rpy=0 0 0 -> xyz=0 0 0.05744 rpy=0 0 0
